File: HUB75-Differential_stepgen/kicad/stepgen_differential_bob.kicad_sch (KiCad schematic)
At the start: 31 parts, among them J1 Conn_02x08_Odd_Even, J2 Conn_02x08_Odd_Even, J3 Conn_02x08_Odd_Even, J4 Screw_Terminal_01x02, J5 RJ45_LED, J6 RJ45_LED, J7 RJ45_LED, SW1 SW_DIP_x03, SW2 SW_DIP_x03, U1 74HC86, U2 74HC86

Commit message: Smaller resistors + production ready
Parts:
- R1, R10, R11, R12, R13, R14, R15, R2, R3, R4, R5, R6, R7, R8, R9: footprint Resistor_SMD:R_2010_5025Metric_Pad1.40x2.65mm_HandSolder -> Resistor_SMD:R_1206_3216Metric_Pad1.30x1.75mm_HandSolder

Commit message: Update to v1.1 after prototype
Parts:
- J1, J2, J3: footprint Connector_PinHeader_2.54mm:PinHeader_2x08_P2.54mm_Vertical -> Connector_IDC:IDC-Header_2x08_P2.54mm_Vertical
- R1, R2, R3, R4, R5, R6: value 290 -> 270
Connections:
- net DRIVE_OK_EXT1: now also J3.1 (Pin_1); no longer J3.3 (Pin_3)
- net DRIVE_OK_EXT2: now also J3.2 (Pin_2); no longer J3.5 (Pin_5)
- net DRIVE_OK_EXT3: now also J3.3 (Pin_3); no longer J3.7 (Pin_7)
- net DRIVE_OK_EXT4: now also J3.5 (Pin_5); no longer J3.1 (Pin_1)
- net DRIVE_OK_EXT5: now also J3.6 (Pin_6); no longer J3.2 (Pin_2)
- net DRIVE_OK_EXT6: now also J3.7 (Pin_7); no longer J3.6 (Pin_6)
Changed lines of the file:
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@@
     )
   )
-  (global_label "DRIVE_OK_EXT6" (shape input) (at 41.91 83.82 0) (fields_autoplaced)
+  (global_label "DRIVE_OK_EXT5" (shape input) (at 41.91 83.82 0) (fields_autoplaced)
     (effects (font (size 1 1)) (justify left))
     (property "Intersheet References" "${INTERSHEET_REFS}" (id 0) (at 55.191 83.7575 0)
@@
     )
   )
-  (global_label "DRIVE_OK_EXT2" (shape input) (at 29.21 83.82 180) (fields_autoplaced)
+  (global_label "DRIVE_OK_EXT4" (shape input) (at 29.21 83.82 180) (fields_autoplaced)
     (effects (font (size 1 1)) (justify right))
     (property "Intersheet References" "${INTERSHEET_REFS}" (id 0) (at 15.929 83.7575 0)
@@
     )
   )
-  (global_label "DRIVE_OK_EXT1" (shape input) (at 29.21 81.28 180) (fields_autoplaced)
+  (global_label "DRIVE_OK_EXT3" (shape input) (at 29.21 81.28 180) (fields_autoplaced)
     (effects (font (size 1 1)) (justify right))
     (property "Intersheet References" "${INTERSHEET_REFS}" (id 0) (at 15.929 81.2175 0)
@@
     )
   )
-  (global_label "DRIVE_OK_EXT4" (shape input) (at 29.21 78.74 180) (fields_autoplaced)
+  (global_label "DRIVE_OK_EXT1" (shape input) (at 29.21 78.74 180) (fields_autoplaced)
     (effects (font (size 1 1)) (justify right))
     (property "Intersheet References" "${INTERSHEET_REFS}" (id 0) (at 15.929 78.6775 0)
@@
     )
   )
-  (global_label "DRIVE_OK_EXT5" (shape input) (at 41.91 78.74 0) (fields_autoplaced)
+  (global_label "DRIVE_OK_EXT2" (shape input) (at 41.91 78.74 0) (fields_autoplaced)
     (effects (font (size 1 1)) (justify left))
     (property "Intersheet References" "${INTERSHEET_REFS}" (id 0) (at 55.191 78.6775 0)
@@
     )
   )
-  (global_label "DRIVE_OK_EXT3" (shape input) (at 29.21 86.36 180) (fields_autoplaced)
+  (global_label "DRIVE_OK_EXT6" (shape input) (at 29.21 86.36 180) (fields_autoplaced)
     (effects (font (size 1 1)) (justify right))
     (property "Intersheet References" "${INTERSHEET_REFS}" (id 0) (at 15.929 86.2975 0)
@@
     (in_bom yes) (on_board yes) (fields_autoplaced)
     (property "Reference" "R1" (id 0) (at 73.66 19.05 90))
-    (property "Value" "290" (id 1) (at 73.66 21.59 90))
+    (property "Value" "270" (id 1) (at 73.66 21.59 90))
     (property "Footprint" "Resistor_SMD:R_1206_3216Metric_Pad1.30x1.75mm_HandSolder" (id 2) (at 73.66 27.178 90)
       (effects (font (size 1.27 1.27)) hide)
@@
     (in_bom yes) (on_board yes) (fields_autoplaced)
     (property "Reference" "R2" (id 0) (at 74.93 36.83 90))
-    (property "Value" "290" (id 1) (at 74.93 39.37 90))
+    (property "Value" "270" (id 1) (at 74.93 39.37 90))
     (property "Footprint" "Resistor_SMD:R_1206_3216Metric_Pad1.30x1.75mm_HandSolder" (id 2) (at 74.93 44.958 90)
       (effects (font (size 1.27 1.27)) hide)
@@
     (in_bom yes) (on_board yes) (fields_autoplaced)
     (property "Reference" "R5" (id 0) (at 74.93 80.01 90))
-    (property "Value" "290" (id 1) (at 74.93 82.55 90))
+    (property "Value" "270" (id 1) (at 74.93 82.55 90))
     (property "Footprint" "Resistor_SMD:R_1206_3216Metric_Pad1.30x1.75mm_HandSolder" (id 2) (at 74.93 88.138 90)
       (effects (font (size 1.27 1.27)) hide)
@@
     (property "Reference" "J3" (id 0) (at 35.56 72.39 0))
     (property "Value" "Conn_02x08_Odd_Even" (id 1) (at 35.56 74.93 0))
-    (property "Footprint" "Connector_PinHeader_2.54mm:PinHeader_2x08_P2.54mm_Vertical" (id 2) (at 34.29 86.36 0)
+    (property "Footprint" "Connector_IDC:IDC-Header_2x08_P2.54mm_Vertical" (id 2) (at 34.29 86.36 0)
       (effects (font (size 1.27 1.27)) hide)
     )
@@
     (property "Reference" "J2" (id 0) (at 35.56 46.99 0))
     (property "Value" "Conn_02x08_Odd_Even" (id 1) (at 35.56 49.53 0))
-    (property "Footprint" "Connector_PinHeader_2.54mm:PinHeader_2x08_P2.54mm_Vertical" (id 2) (at 34.29 60.96 0)
+    (property "Footprint" "Connector_IDC:IDC-Header_2x08_P2.54mm_Vertical" (id 2) (at 34.29 60.96 0)
       (effects (font (size 1.27 1.27)) hide)
     )
@@
     (in_bom yes) (on_board yes) (fields_autoplaced)
     (property "Reference" "R6" (id 0) (at 74.93 97.79 90))
-    (property "Value" "290" (id 1) (at 74.93 100.33 90))
+    (property "Value" "270" (id 1) (at 74.93 100.33 90))
     (property "Footprint" "Resistor_SMD:R_1206_3216Metric_Pad1.30x1.75mm_HandSolder" (id 2) (at 74.93 105.918 90)
       (effects (font (size 1.27 1.27)) hide)
@@
     (in_bom yes) (on_board yes) (fields_autoplaced)
     (property "Reference" "R3" (id 0) (at 74.93 49.53 90))
-    (property "Value" "290" (id 1) (at 74.93 52.07 90))
+    (property "Value" "270" (id 1) (at 74.93 52.07 90))
     (property "Footprint" "Resistor_SMD:R_1206_3216Metric_Pad1.30x1.75mm_HandSolder" (id 2) (at 74.93 57.658 90)
       (effects (font (size 1.27 1.27)) hide)
@@
     (in_bom yes) (on_board yes) (fields_autoplaced)
     (property "Reference" "R4" (id 0) (at 74.93 67.31 90))
-    (property "Value" "290" (id 1) (at 74.93 69.85 90))
+    (property "Value" "270" (id 1) (at 74.93 69.85 90))
     (property "Footprint" "Resistor_SMD:R_1206_3216Metric_Pad1.30x1.75mm_HandSolder" (id 2) (at 74.93 75.438 90)
       (effects (font (size 1.27 1.27)) hide)
@@
     (property "Reference" "J1" (id 0) (at 35.56 19.05 0))
     (property "Value" "Conn_02x08_Odd_Even" (id 1) (at 35.56 21.59 0))
-    (property "Footprint" "Connector_PinHeader_2.54mm:PinHeader_2x08_P2.54mm_Vertical" (id 2) (at 34.29 33.02 0)
+    (property "Footprint" "Connector_IDC:IDC-Header_2x08_P2.54mm_Vertical" (id 2) (at 34.29 33.02 0)
       (effects (font (size 1.27 1.27)) hide)
     )
@@
     )
     (path "/c8fd9dd3-06ad-4146-9239-0065013959ef"
-      (reference "J1") (unit 1) (value "Conn_02x08_Odd_Even") (footprint "Connector_PinHeader_2.54mm:PinHeader_2x08_P2.54mm_Vertical")
+      (reference "J1") (unit 1) (value "Conn_02x08_Odd_Even") (footprint "Connector_IDC:IDC-Header_2x08_P2.54mm_Vertical")
     )
     (path "/719303cc-9ddf-4f19-9751-b8db3875f499"
-      (reference "J2") (unit 1) (value "Conn_02x08_Odd_Even") (footprint "Connector_PinHeader_2.54mm:PinHeader_2x08_P2.54mm_Vertical")
+      (reference "J2") (unit 1) (value "Conn_02x08_Odd_Even") (footprint "Connector_IDC:IDC-Header_2x08_P2.54mm_Vertical")
     )
     (path "/5e55078b-97af-4c80-838b-eaf4f630bb7a"
-      (reference "J3") (unit 1) (value "Conn_02x08_Odd_Even") (footprint "Connector_PinHeader_2.54mm:PinHeader_2x08_P2.54mm_Vertical")
+      (reference "J3") (unit 1) (value "Conn_02x08_Odd_Even") (footprint "Connector_IDC:IDC-Header_2x08_P2.54mm_Vertical")
     )
     (path "/e7350447-059e-4528-8aab-e44104118b00"
@@
     )
     (path "/24234257-d365-4c66-89b5-092b815cbaea"
-      (reference "R1") (unit 1) (value "290") (footprint "Resistor_SMD:R_1206_3216Metric_Pad1.30x1.75mm_HandSolder")
+      (reference "R1") (unit 1) (value "270") (footprint "Resistor_SMD:R_1206_3216Metric_Pad1.30x1.75mm_HandSolder")
     )
     (path "/3ef498b3-0fb1-4e20-ac79-8153cbef4a74"
-      (reference "R2") (unit 1) (value "290") (footprint "Resistor_SMD:R_1206_3216Metric_Pad1.30x1.75mm_HandSolder")
+      (reference "R2") (unit 1) (value "270") (footprint "Resistor_SMD:R_1206_3216Metric_Pad1.30x1.75mm_HandSolder")
     )
     (path "/784b0d57-4676-4b4b-976a-04eb228df8eb"
-      (reference "R3") (unit 1) (value "290") (footprint "Resistor_SMD:R_1206_3216Metric_Pad1.30x1.75mm_HandSolder")
+      (reference "R3") (unit 1) (value "270") (footprint "Resistor_SMD:R_1206_3216Metric_Pad1.30x1.75mm_HandSolder")
     )
     (path "/aa2ce174-d029-45da-839f-64a40b59c884"
-      (reference "R4") (unit 1) (value "290") (footprint "Resistor_SMD:R_1206_3216Metric_Pad1.30x1.75mm_HandSolder")
+      (reference "R4") (unit 1) (value "270") (footprint "Resistor_SMD:R_1206_3216Metric_Pad1.30x1.75mm_HandSolder")
     )
     (path "/595efaee-6b86-4c6a-afdf-efc352080aba"
-      (reference "R5") (unit 1) (value "290") (footprint "Resistor_SMD:R_1206_3216Metric_Pad1.30x1.75mm_HandSolder")
+      (reference "R5") (unit 1) (value "270") (footprint "Resistor_SMD:R_1206_3216Metric_Pad1.30x1.75mm_HandSolder")
     )
     (path "/75fff4a6-e227-41ed-8353-ce7adf832eb7"
-      (reference "R6") (unit 1) (value "290") (footprint "Resistor_SMD:R_1206_3216Metric_Pad1.30x1.75mm_HandSolder")
+      (reference "R6") (unit 1) (value "270") (footprint "Resistor_SMD:R_1206_3216Metric_Pad1.30x1.75mm_HandSolder")
     )
     (path "/c51de39d-fa75-4ec5-90f8-9c16896bd560"
