File: HUB75-Sinking_input/kicad/HUB75-Sinking_input.kicad_pcb (KiCad board)
At the start: 2 copper layers, 85 x 56 mm, 81 parts, among them J1 Conn_01x03_Male, J10 Conn_01x03_Male, J11 Conn_01x03_Male, J12 Conn_01x03_Male, J2 Conn_01x03_Male, J3 Conn_01x03_Male, J4 Conn_01x03_Male, J5 Conn_01x03_Male, J6 Conn_01x03_Male, J7 Conn_01x03_Male, J8 Conn_01x03_Male, J9 Conn_01x03_Male, Q1 AO3401A, Q10 2N7002, Q11 2N7002, Q12 2N7002, Q13 2N7002, Q14 2N7002, Q2 2N7002, Q3 2N7002, Q4 2N7002, Q5 2N7002, Q6 2N7002, Q7 2N7002, Q8 2N7002, Q9 2N7002, U1 CL2N8-G, U2 LTV-827, U3 LTV-827, U4 LTV-827, U5 LTV-827, U6 LTV-827, U7 LTV-827

Commit message: Version for prototype
Parts:
- added JP1: Jumper_2_Open, Jumper:SolderJumper-2_P1.3mm_Open_TrianglePad1.0x1.5mm, B.Cu at (106.7, 64.8)
- D1: footprint Diode_SMD:D_SOD-123 -> Diode_SMD:D_SOT-23_ANK
- HUB75-1, HUB75-2: footprint Connector_PinHeader_2.54mm:PinHeader_2x08_P2.54mm_Vertical -> Connector_IDC:IDC-Header_2x08_P2.54mm_Vertical
- R11, R13, R15, R17, R19, R21, R23, R25, R3, R5, R7, R9: moved to B.Cu
- moved G*** 71.7 mm to (45.2, 78.0)
- moved HUB75-2 8.95 mm to (80.3, 34.0)
- moved R1 3.18 mm to (113.0, 55.9), turned to 90 degrees
- moved HUB75-1 2.28 mm to (45.5, 34.0)
- moved C1 1.02 mm to (110.2, 55.9), turned to 90 degrees
- moved D1 0.76 mm to (106.4, 58.4), turned to 180 degrees
- renumbered PWR2 to PWR1, PWR1 to PWR2
Routing:
- net GPIO2-3: track 25.1 -> 13.2 mm
- net GPIO2-6: track 27.5 -> 15.7 mm
- net GPIO1-1: track 18.1 -> 10.9 mm
- net GPIO1-2: track 24.5 -> 17.4 mm
- net GPIO2-5: track 34.3 -> 28.5 mm
- net GPIO2-2: track 14.5 -> 18.7 mm
- net GPIO2-4: track 15.1 -> 11.4 mm
- net VDD: track 182.9 -> 186.0 mm
- net GPIO1-3: track 13.7 -> 11.0 mm
- net Net-(PWR1-Pad2): track 5.92 -> 8.31 mm
- net GPIO1-6: track 12.1 -> 14.4 mm
- net GPIO1-5: track 23.4 -> 22.3 mm
- net Net-(C1-Pad1): track 7.22 -> 8.09 mm
- net GPIO1-4: track 11.8 -> 12.4 mm
