File: HUB75-Sinking_input/kicad/HUB75-Sinking_input.kicad_sch (KiCad schematic)
At the start: 10 parts, among them Q1 AO3401A, Q2 2N7002, U1 CL2N8-G

Commit message: Version for prototype
Parts:
- added JP1: Jumper_2_Open, Jumper:SolderJumper-2_P1.3mm_Open_TrianglePad1.0x1.5mm, symbol Jumper:Jumper_2_Open
- D1: footprint Diode_SMD:D_SOD-123 -> Diode_SMD:D_SOT-23_ANK
- HUB75-1, HUB75-2: footprint Connector_PinHeader_2.54mm:PinHeader_2x08_P2.54mm_Vertical -> Connector_IDC:IDC-Header_2x08_P2.54mm_Vertical
- gave numbers to parts that had none: 1
Connections:
- net VDD: now also JP1.2 (B)
- net at PWR1.2 (Pin_2), Q1.2 (S): now also JP1.1 (A)
Changed lines of the file:
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@@
   (junction (at 107.95 184.15) (diameter 0) (color 0 0 0 0)
   )
+  (junction (at 36.83 173.99) (diameter 0) (color 0 0 0 0)
+  )
   (junction (at 44.45 189.23) (diameter 0) (color 0 0 0 0)
   )
@@
     (stroke (width 0) (type default) (color 0 0 0 0))
   )
+  (wire (pts (xy 53.34 166.37) (xy 53.34 173.99))
+    (stroke (width 0) (type default) (color 0 0 0 0))
+  )
   (polyline (pts (xy 83.82 158.75) (xy 83.82 196.85))
     (stroke (width 0) (type default) (color 0 0 0 0))
@@
     (stroke (width 0) (type default) (color 0 0 0 0))
   )
+  (wire (pts (xy 49.53 166.37) (xy 53.34 166.37))
+    (stroke (width 0) (type default) (color 0 0 0 0))
+  )
   (polyline (pts (xy 133.35 158.75) (xy 133.35 196.85))
     (stroke (width 0) (type default) (color 0 0 0 0))
@@
     (stroke (width 0) (type default) (color 0 0 0 0))
   )
+  (wire (pts (xy 39.37 166.37) (xy 36.83 166.37))
+    (stroke (width 0) (type default) (color 0 0 0 0))
+  )
   (wire (pts (xy 123.19 63.5) (xy 125.73 63.5))
     (stroke (width 0) (type default) (color 0 0 0 0))
@@
     (stroke (width 0) (type default) (color 0 0 0 0))
   )
+  (wire (pts (xy 36.83 173.99) (xy 39.37 173.99))
+    (stroke (width 0) (type default) (color 0 0 0 0))
+  )
   (wire (pts (xy 44.45 189.23) (xy 53.34 189.23))
     (stroke (width 0) (type default) (color 0 0 0 0))
@@
     (stroke (width 0) (type default) (color 0 0 0 0))
   )
-  (wire (pts (xy 33.02 173.99) (xy 39.37 173.99))
+  (wire (pts (xy 33.02 173.99) (xy 36.83 173.99))
     (stroke (width 0) (type default) (color 0 0 0 0))
   )
   (wire (pts (xy 177.8 38.1) (xy 180.34 38.1))
+    (stroke (width 0) (type default) (color 0 0 0 0))
+  )
+  (wire (pts (xy 36.83 166.37) (xy 36.83 173.99))
     (stroke (width 0) (type default) (color 0 0 0 0))
   )
@@
     (pin "2")
   )
+  (symbol (lib_id "Jumper:Jumper_2_Open") (at 44.45 166.37 0) (unit 1)
+    (in_bom yes) (on_board yes) (fields_autoplaced)
+    (property "Reference" "JP1" (id 0) (at 44.45 160.02 0))
+    (property "Value" "Jumper_2_Open" (id 1) (at 44.45 162.56 0))
+    (property "Footprint" "Jumper:SolderJumper-2_P1.3mm_Open_TrianglePad1.0x1.5mm" (id 2) (at 44.45 166.37 0)
+      (effects (font (size 1.27 1.27)) hide)
+    )
+    (property "Datasheet" "~" (id 3) (at 44.45 166.37 0)
+      (effects (font (size 1.27 1.27)) hide)
+    )
+    (pin "1")
+    (pin "2")
+  )
   (symbol (lib_id "power:GND") (at 33.02 133.35 0) (unit 1)
     (in_bom yes) (on_board yes) (fields_autoplaced)
-    (property "Reference" "#PWR?" (id 0) (at 33.02 139.7 0)
+    (property "Reference" "#PWR0113" (id 0) (at 33.02 139.7 0)
       (effects (font (size 1.27 1.27)) hide)
     )
@@
     (property "Reference" "HUB75-2" (id 0) (at 36.83 52.07 0))
     (property "Value" "Conn_02x08_Odd_Even" (id 1) (at 36.83 54.61 0))
-    (property "Footprint" "Connector_PinHeader_2.54mm:PinHeader_2x08_P2.54mm_Vertical" (id 2) (at 35.56 66.04 0)
+    (property "Footprint" "Connector_IDC:IDC-Header_2x08_P2.54mm_Vertical" (id 2) (at 35.56 66.04 0)
       (effects (font (size 1.27 1.27)) hide)
     )
@@
       (effects (font (size 1.27 1.27)) (justify left))
     )
-    (property "Footprint" "Diode_SMD:D_SOD-123" (id 2) (at 53.34 177.8 0)
+    (property "Footprint" "Diode_SMD:D_SOT-23_ANK" (id 2) (at 53.34 177.8 0)
       (effects (font (size 1.27 1.27)) hide)
     )
@@
   (symbol (lib_id "power:+5V") (at 39.37 130.81 270) (unit 1)
     (in_bom yes) (on_board yes) (fields_autoplaced)
-    (property "Reference" "#PWR?" (id 0) (at 35.56 130.81 0)
+    (property "Reference" "#PWR0114" (id 0) (at 35.56 130.81 0)
       (effects (font (size 1.27 1.27)) hide)
     )
@@
   (symbol (lib_id "Connector:Screw_Terminal_01x02") (at 27.94 133.35 180) (unit 1)
     (in_bom yes) (on_board yes) (fields_autoplaced)
-    (property "Reference" "PWR?" (id 0) (at 27.94 124.46 0))
+    (property "Reference" "PWR2" (id 0) (at 27.94 124.46 0))
     (property "Value" "Screw_Terminal_01x02" (id 1) (at 27.94 127 0))
     (property "Footprint" "TerminalBlock_Phoenix:TerminalBlock_Phoenix_PT-1,5-2-3.5-H_1x02_P3.50mm_Horizontal" (id 2) (at 27.94 133.35 0)
@@
     (property "Reference" "HUB75-1" (id 0) (at 36.83 17.78 0))
     (property "Value" "Conn_02x08_Odd_Even" (id 1) (at 36.83 20.32 0))
-    (property "Footprint" "Connector_PinHeader_2.54mm:PinHeader_2x08_P2.54mm_Vertical" (id 2) (at 35.56 31.75 0)
+    (property "Footprint" "Connector_IDC:IDC-Header_2x08_P2.54mm_Vertical" (id 2) (at 35.56 31.75 0)
       (effects (font (size 1.27 1.27)) hide)
     )
@@
     )
     (path "/24a022b0-6c29-4b10-8b4d-1b85124e46b5"
-      (reference "#PWR?") (unit 1) (value "GND") (footprint "")
+      (reference "#PWR0113") (unit 1) (value "GND") (footprint "")
     )
     (path "/8c916ec3-8533-4f7b-bec7-e24b20fb4c88"
-      (reference "#PWR?") (unit 1) (value "+5V") (footprint "")
+      (reference "#PWR0114") (unit 1) (value "+5V") (footprint "")
     )
     (path "/d88958ac-68cd-4955-a63f-0eaa329dec86"
@@
     )
     (path "/477892a1-722e-4cda-bb6c-fcdb8ba5f93e"
-      (reference "D1") (unit 1) (value "D_Zener") (footprint "Diode_SMD:D_SOD-123")
+      (reference "D1") (unit 1) (value "D_Zener") (footprint "Diode_SMD:D_SOT-23_ANK")
     )
     (path "/4beab297-7e95-4e96-a8ef-c9404d55c3ef/4d24efbc-f4ce-4aeb-b127-5ff3e27b027a"
@@
     )
     (path "/da85e218-28f5-4e04-9ae0-77a4ed9bdc04"
-      (reference "HUB75-1") (unit 1) (value "Conn_02x08_Odd_Even") (footprint "Connector_PinHeader_2.54mm:PinHeader_2x08_P2.54mm_Vertical")
+      (reference "HUB75-1") (unit 1) (value "Conn_02x08_Odd_Even") (footprint "Connector_IDC:IDC-Header_2x08_P2.54mm_Vertical")
     )
     (path "/2c8a6197-c8f2-4731-a9bd-21ee0dc98785"
-      (reference "HUB75-2") (unit 1) (value "Conn_02x08_Odd_Even") (footprint "Connector_PinHeader_2.54mm:PinHeader_2x08_P2.54mm_Vertical")
+      (reference "HUB75-2") (unit 1) (value "Conn_02x08_Odd_Even") (footprint "Connector_IDC:IDC-Header_2x08_P2.54mm_Vertical")
     )
     (path "/4beab297-7e95-4e96-a8ef-c9404d55c3ef/1ce2fc39-63eb-4c3b-a684-88c7a188fecd"
@@
       (reference "J12") (unit 1) (value "Conn_01x03_Male") (footprint "Connector_JST:JST_XH_B3B-XH-A_1x03_P2.50mm_Vertical")
     )
+    (path "/1974c726-def2-42f6-bccb-1a0f7b6515d7"
+      (reference "JP1") (unit 1) (value "Jumper_2_Open") (footprint "Jumper:SolderJumper-2_P1.3mm_Open_TrianglePad1.0x1.5mm")
+    )
     (path "/9f80220c-1612-4589-b9ca-a5579617bdb8"
       (reference "PWR1") (unit 1) (value "Screw_Terminal_01x02") (footprint "TerminalBlock_Phoenix:TerminalBlock_Phoenix_PT-1,5-2-3.5-H_1x02_P3.50mm_Horizontal")
     )
     (path "/bb4d6457-fabc-4955-99fd-f7563197de92"
-      (reference "PWR?") (unit 1) (value "Screw_Terminal_01x02") (footprint "TerminalBlock_Phoenix:TerminalBlock_Phoenix_PT-1,5-2-3.5-H_1x02_P3.50mm_Horizontal")
+      (reference "PWR2") (unit 1) (value "Screw_Terminal_01x02") (footprint "TerminalBlock_Phoenix:TerminalBlock_Phoenix_PT-1,5-2-3.5-H_1x02_P3.50mm_Horizontal")
     )
     (path "/e5203297-b913-4288-a576-12a92185cb52"
