File: HUB75-Sinking_input/kicad/optocoupler_channel.kicad_sch (KiCad schematic)
At the start: 12 parts, among them J7 Conn_01x03_Male, J8 Conn_01x03_Male, Q10 2N7002, Q9 2N7002, U5 LTV-827

Commit message: Version for prototype
Parts:
- renumbered D8 to D12, D9 to D13, J7 to J11, J8 to J12, Q9 to Q13, Q10 to Q14, R14 to R22, R15 to R23, R16 to R24, R17 to R25, U5 to U7
Changed lines of the file:
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@@
   (symbol (lib_id "Transistor_FET:2N7002") (at 46.99 102.87 270) (mirror x)
     (in_bom yes) (on_board yes) (fields_autoplaced)
-    (property "Reference" "Q10" (id 0) (at 46.99 92.71 90))
+    (property "Reference" "Q14" (id 0) (at 46.99 92.71 90))
     (property "Value" "2N7002" (id 1) (at 46.99 95.25 90))
     (property "Footprint" "Package_TO_SOT_SMD:SOT-23" (id 2) (at 45.085 97.79 0)
@@
   (symbol (lib_id "Isolator:LTV-827") (at 66.04 86.36 0)
     (in_bom yes) (on_board yes) (fields_autoplaced)
-    (property "Reference" "U5" (id 0) (at 66.04 77.47 0))
+    (property "Reference" "U7" (id 0) (at 66.04 77.47 0))
     (property "Value" "LTV-827" (id 1) (at 66.04 80.01 0))
     (property "Footprint" "Package_DIP:DIP-8_W7.62mm" (id 2) (at 60.96 91.44 0)
@@
   (symbol (lib_id "power:VDD") (at 39.37 81.28 0)
     (in_bom yes) (on_board yes) (fields_autoplaced)
-    (property "Reference" "#PWR0108" (id 0) (at 39.37 85.09 0)
+    (property "Reference" "#PWR0112" (id 0) (at 39.37 85.09 0)
       (effects (font (size 1.27 1.27)) hide)
     )
@@
   (symbol (lib_id "Connector:Conn_01x03_Male") (at 34.29 31.75 0)
     (in_bom yes) (on_board yes)
-    (property "Reference" "J7" (id 0) (at 34.925 24.13 0))
+    (property "Reference" "J11" (id 0) (at 34.925 24.13 0))
     (property "Value" "Conn_01x03_Male" (id 1) (at 34.925 26.67 0))
     (property "Footprint" "Connector_JST:JST_XH_B3B-XH-A_1x03_P2.50mm_Vertical" (id 2) (at 34.29 31.75 0)
@@
   (symbol (lib_id "Isolator:LTV-827") (at 66.04 34.29 0)
     (in_bom yes) (on_board yes) (fields_autoplaced)
-    (property "Reference" "U5" (id 0) (at 66.04 25.4 0))
+    (property "Reference" "U7" (id 0) (at 66.04 25.4 0))
     (property "Value" "LTV-827" (id 1) (at 66.04 27.94 0))
     (property "Footprint" "Package_DIP:DIP-8_W7.62mm" (id 2) (at 60.96 39.37 0)
@@
   (symbol (lib_id "Device:R") (at 73.66 92.71 0)
     (in_bom yes) (on_board yes) (fields_autoplaced)
-    (property "Reference" "R17" (id 0) (at 76.2 91.4399 0)
+    (property "Reference" "R25" (id 0) (at 76.2 91.4399 0)
       (effects (font (size 1.27 1.27)) (justify left))
     )
@@
   (symbol (lib_id "Connector:Conn_01x03_Male") (at 34.29 83.82 0)
     (in_bom yes) (on_board yes)
-    (property "Reference" "J8" (id 0) (at 34.925 76.2 0))
+    (property "Reference" "J12" (id 0) (at 34.925 76.2 0))
     (property "Value" "Conn_01x03_Male" (id 1) (at 34.925 78.74 0))
     (property "Footprint" "Connector_JST:JST_XH_B3B-XH-A_1x03_P2.50mm_Vertical" (id 2) (at 34.29 83.82 0)
@@
   (symbol (lib_id "Transistor_FET:2N7002") (at 46.99 50.8 270) (mirror x)
     (in_bom yes) (on_board yes) (fields_autoplaced)
-    (property "Reference" "Q9" (id 0) (at 46.99 40.64 90))
+    (property "Reference" "Q13" (id 0) (at 46.99 40.64 90))
     (property "Value" "2N7002" (id 1) (at 46.99 43.18 90))
     (property "Footprint" "Package_TO_SOT_SMD:SOT-23" (id 2) (at 45.085 45.72 0)
@@
   (symbol (lib_id "Device:LED_Small") (at 55.88 36.83 0)
     (in_bom yes) (on_board yes)
-    (property "Reference" "D8" (id 0) (at 55.88 39.37 0))
+    (property "Reference" "D12" (id 0) (at 55.88 39.37 0))
     (property "Value" "LED_Small" (id 1) (at 55.88 41.91 0))
     (property "Footprint" "LED_SMD:LED_1206_3216Metric_Pad1.42x1.75mm_HandSolder" (id 2) (at 55.88 36.83 90)
@@
   (symbol (lib_id "Device:R") (at 46.99 36.83 90)
     (in_bom yes) (on_board yes)
-    (property "Reference" "R14" (id 0) (at 46.99 34.29 90))
+    (property "Reference" "R22" (id 0) (at 46.99 34.29 90))
     (property "Value" "R" (id 1) (at 46.99 33.02 90)
       (effects (font (size 1.27 1.27)) hide)
@@
   (symbol (lib_id "Device:R") (at 73.66 40.64 0)
     (in_bom yes) (on_board yes) (fields_autoplaced)
-    (property "Reference" "R15" (id 0) (at 76.2 39.3699 0)
+    (property "Reference" "R23" (id 0) (at 76.2 39.3699 0)
       (effects (font (size 1.27 1.27)) (justify left))
     )
@@
   (symbol (lib_id "power:GND") (at 73.66 44.45 0)
     (in_bom yes) (on_board yes)
-    (property "Reference" "#PWR031" (id 0) (at 73.66 50.8 0)
+    (property "Reference" "#PWR047" (id 0) (at 73.66 50.8 0)
       (effects (font (size 1.27 1.27)) hide)
     )
@@
   (symbol (lib_id "Device:R") (at 46.99 88.9 90)
     (in_bom yes) (on_board yes)
-    (property "Reference" "R16" (id 0) (at 46.99 86.36 90))
+    (property "Reference" "R24" (id 0) (at 46.99 86.36 90))
     (property "Value" "R" (id 1) (at 46.99 85.09 90)
       (effects (font (size 1.27 1.27)) hide)
@@
   (symbol (lib_id "power:GND") (at 73.66 96.52 0)
     (in_bom yes) (on_board yes) (fields_autoplaced)
-    (property "Reference" "#PWR035" (id 0) (at 73.66 102.87 0)
+    (property "Reference" "#PWR051" (id 0) (at 73.66 102.87 0)
       (effects (font (size 1.27 1.27)) hide)
     )
@@
   (symbol (lib_id "power:+5V") (at 73.66 83.82 0)
     (in_bom yes) (on_board yes) (fields_autoplaced)
-    (property "Reference" "#PWR034" (id 0) (at 73.66 87.63 0)
+    (property "Reference" "#PWR050" (id 0) (at 73.66 87.63 0)
       (effects (font (size 1.27 1.27)) hide)
     )
@@
   (symbol (lib_id "power:GNDD") (at 39.37 50.8 0)
     (in_bom yes) (on_board yes)
-    (property "Reference" "#PWR032" (id 0) (at 39.37 57.15 0)
+    (property "Reference" "#PWR048" (id 0) (at 39.37 57.15 0)
       (effects (font (size 1.27 1.27)) hide)
     )
@@
   (symbol (lib_id "power:VDD") (at 39.37 29.21 0)
     (in_bom yes) (on_board yes) (fields_autoplaced)
-    (property "Reference" "#PWR0107" (id 0) (at 39.37 33.02 0)
+    (property "Reference" "#PWR0111" (id 0) (at 39.37 33.02 0)
       (effects (font (size 1.27 1.27)) hide)
     )
@@
   (symbol (lib_id "Device:LED_Small") (at 55.88 88.9 0)
     (in_bom yes) (on_board yes)
-    (property "Reference" "D9" (id 0) (at 55.88 91.44 0))
+    (property "Reference" "D13" (id 0) (at 55.88 91.44 0))
     (property "Value" "LED_Small" (id 1) (at 55.88 93.98 0))
     (property "Footprint" "LED_SMD:LED_1206_3216Metric_Pad1.42x1.75mm_HandSolder" (id 2) (at 55.88 88.9 90)
@@
   (symbol (lib_id "power:+5V") (at 73.66 31.75 0)
     (in_bom yes) (on_board yes) (fields_autoplaced)
-    (property "Reference" "#PWR030" (id 0) (at 73.66 35.56 0)
+    (property "Reference" "#PWR046" (id 0) (at 73.66 35.56 0)
       (effects (font (size 1.27 1.27)) hide)
     )
@@
   (symbol (lib_id "power:GNDD") (at 39.37 102.87 0)
     (in_bom yes) (on_board yes)
-    (property "Reference" "#PWR036" (id 0) (at 39.37 109.22 0)
-      (effects (font (size 1.27 1.27)) hide)
-    )
+    (property "Reference" "#PWR052" (id 0) (at 39.37 109.22 0)
+      (effects (font (size 1.27 1.27)) hide)
+    )
